Commit message: Fix leg model

File: src/robot/arm_description/urdf/leg.urdf (robot description, URDF)
Before this commit: robot mulinex, 7 links, 6 joints
Links:
- removed link world
- added link world_link, mass 1000.0; collision box size=10 10 0.01
Joints:
- joint base_to_world: parent world -> world_link

File: src/robot/arm_description/urdf/leg.xacro (robot description, xacro)
@@ -10,5 +10,11 @@
     <xacro:property name="joint_2" value="0.0" />
     <xacro:property name="joint_3" value="0.0" />
-    <link name="world">
+    <link name="world_link">
+        <visual>
+            <material name="white" />
+            <geometry>
+                <box size="10 10 0.01" />
+            </geometry>
+        </visual>
         <collision>
             <geometry>
@@ -22,5 +28,5 @@
     </link>
     <joint name="base_to_world" type="prismatic">
-        <parent link="world" />
+        <parent link="world_link" />
         <child link="base_link" />
         <origin xyz="0 0 0.6" rpy="0 0 0" />
