Commit message: First commit of leg controller

File: src/robot/arm_description/urdf/leg.xacro (robot description, xacro)
@@ -24,5 +24,5 @@
         <parent link="world" />
         <child link="base_link" />
-        <origin xyz="0 0 0.75" rpy="0 0 0" />
+        <origin xyz="0 0 0.6" rpy="0 0 0" />
         <axis xyz="0 0 1" />
         <limit effort="100.0" velocity="100.0" lower="-1.0" upper="1.0" />

Commit message: Small changes

File: src/robot/arm_description/urdf/leg.xacro (robot description, xacro)
@@ -11,10 +11,10 @@
     <xacro:property name="joint_3" value="0.0" />
     <link name="world_link">
-        <visual>
+        <!-- <visual>
             <material name="white" />
             <geometry>
                 <box size="10 10 0.01" />
             </geometry>
-        </visual>
+        </visual> -->
         <collision>
             <geometry>
