Commit message: Add PD controller with slider controlled reference

File: src/robot/arm_description/urdf/arm_gazebo.xacro (robot description, xacro)
@@ -18,7 +18,7 @@
             <plugin>gz_ros2_control/GazeboSimSystem</plugin>
         </hardware>
-        <xacro:ros2_control_joint joint_name="JOINT_1" effort_lim="10" initial_value="0.0"></xacro:ros2_control_joint>
-        <xacro:ros2_control_joint joint_name="JOINT_2" effort_lim="10" initial_value="0.0"></xacro:ros2_control_joint>
-        <xacro:ros2_control_joint joint_name="JOINT_3" effort_lim="10" initial_value="0.0"></xacro:ros2_control_joint>
+        <xacro:ros2_control_joint joint_name="JOINT_1" effort_lim="10" initial_value="-0.6"></xacro:ros2_control_joint>
+        <xacro:ros2_control_joint joint_name="JOINT_2" effort_lim="10" initial_value=" 0.6"></xacro:ros2_control_joint>
+        <xacro:ros2_control_joint joint_name="JOINT_3" effort_lim="10" initial_value=" 0.6"></xacro:ros2_control_joint>
     </ros2_control>
     <gazebo>

File: src/robot/arm_description/urdf/leg.xacro (robot description, xacro)
@@ -30,5 +30,5 @@
         <parent link="world_link" />
         <child link="base_link" />
-        <origin xyz="0 0 0.6" rpy="0 0 0" />
+        <origin xyz="0 0 0.525" rpy="0 0 0" />
         <axis xyz="0 0 1" />
         <limit effort="100.0" velocity="100.0" lower="-1.0" upper="1.0" />
