Commit message: Add simulation in Gazebo

File: src/robot/arm_description/urdf/arm.xacro (robot description, xacro)
@@ -10,4 +10,20 @@
     <xacro:property name="joint_2" value="0.0" />
     <xacro:property name="joint_3" value="0.0" />
+    <link name="world">
+        <collision>
+            <geometry>
+                <box size="10 10 0.01" />
+            </geometry>
+        </collision>
+        <inertial>
+            <mass value="1000.0" />
+            <inertia ixx="100.0" ixy="0.0" ixz="0.0" iyy="100.0" iyz="0.0" izz="100.0" />
+        </inertial>
+    </link>
+    <joint name="base_to_world" type="fixed">
+        <parent link="world" />
+        <child link="base_link" />
+        <origin xyz="0 0 1" rpy="0 0 0" />
+    </joint>
     <link name="${jnt_prefix}base_link"></link>
     <joint name="JOINT_0" type="fixed">
@@ -33,45 +49,3 @@
         jnt_pref="${jnt_prefix}"
         simplify_meshes="${simplify_meshes_lower_leg}" />
-    <xacro:if value="${use_gazebo}">
-        <gazebo reference="base_link">
-            <material>Gazebo/White</material>
-        </gazebo>
-        <ros2_control name="GazeboSystem" type="system">
-            <hardware>
-                <plugin>gazebo_ros2_control/GazeboSystem</plugin>
-            </hardware>
-            <joint name="JOINT_1">
-                <command_interface name="effort" />
-                <state_interface name="position">
-                    <param name="initial_value">-${joint_1}</param>
-                </state_interface>
-                <state_interface name="velocity">
-                    <param name="initial_value">0.0</param>
-                </state_interface>
-                <state_interface name="effort" />
-            </joint>
-            <joint name="JOINT_2">
-                <command_interface name="effort" />
-                <state_interface name="position">
-                    <param name="initial_value">${joint_2}</param>
-                </state_interface>
-                <state_interface name="velocity">
-                    <param name="initial_value">0.0</param>
-                </state_interface>
-                <state_interface name="effort" />
-            </joint>
-            <joint name="JOINT_3">
-                <command_interface name="effort" />
-                <state_interface name="position">
-                    <param name="initial_value">${joint_3}</param>
-                </state_interface>
-                <state_interface name="velocity">
-                    <param name="initial_value">0.0</param>
-                </state_interface>
-                <state_interface name="effort" />
-            </joint>
-        </ros2_control>
-    </xacro:if>
-    <xacro:unless value="${use_gazebo}">
-    </xacro:unless>
 </robot>

Commit message: Change camera orientation

File: src/robot/arm_description/urdf/arm.xacro (robot description, xacro)
@@ -24,5 +24,5 @@
         <parent link="world" />
         <child link="base_link" />
-        <origin xyz="0 0 1" rpy="0 0 0" />
+        <origin xyz="0 0 0.75" rpy="0 0 0" />
     </joint>
     <link name="${jnt_prefix}base_link"></link>

Commit message: Add arg to arm xacro

File: src/robot/arm_description/urdf/arm.xacro (robot description, xacro)
@@ -1,8 +1,5 @@
 <?xml version="1.0"?>
 <robot name="mulinex" xmlns:xacro="http://ros.org/wiki/xacro">
-    <xacro:include filename="$(find arm_description)/urdf/links.xacro" />
-    <xacro:include filename="$(find arm_description)/urdf/material.xacro" />
-    <xacro:include filename="$(find arm_description)/urdf/arm_gazebo.xacro" />
-    <xacro:property name="use_gazebo" value="true" />
+    <xacro:arg name="use_gazebo" default="true" />
     <xacro:property name="simplify_meshes_lower_leg" value="false"/>
     <xacro:property name="jnt_prefix" value="" />
@@ -10,4 +7,9 @@
     <xacro:property name="joint_2" value="0.0" />
     <xacro:property name="joint_3" value="0.0" />
+    <xacro:include filename="$(find arm_description)/urdf/links.xacro" />
+    <xacro:include filename="$(find arm_description)/urdf/material.xacro" />
+    <xacro:if value="$(arg use_gazebo)">
+        <xacro:include filename="$(find arm_description)/urdf/arm_gazebo.xacro" />
+    </xacro:if>
     <link name="world">
         <collision>
@@ -34,17 +36,17 @@
     <xacro:module
         prefix="1"
-        gazebo="${use_gazebo}"
+        gazebo="$(arg use_gazebo)"
         jnt_pref="${jnt_prefix}" />
     <xacro:module
         prefix="2"
-        gazebo="${use_gazebo}"
+        gazebo="$(arg use_gazebo)"
         jnt_pref="${jnt_prefix}" />
     <xacro:module
         prefix="3"
-        gazebo="${use_gazebo}"
+        gazebo="$(arg use_gazebo)"
         jnt_pref="${jnt_prefix}" />
     <xacro:module_ee
         prefix="4"
-        gazebo="${use_gazebo}"
+        gazebo="$(arg use_gazebo)"
         jnt_pref="${jnt_prefix}"
         simplify_meshes="${simplify_meshes_lower_leg}" />
