Commit message: Update meshes paths

File: src/robot/arm_description/urdf/arm.urdf (robot description, URDF)
Before this commit: robot mulinex, 6 links, 5 joints
Links:
- link MODULE_1: geometry collision box size=0.269 0.057 0.060; visual mesh filename=package://arm_description/meshes/Module_right_front.stl
- link MODULE_2: geometry collision box size=0.269 0.057 0.060; visual mesh filename=package://arm_description/meshes/Module_right_front.stl
- link MODULE_3: geometry collision box size=0.269 0.057 0.060; visual mesh filename=package://arm_description/meshes/Module_right_front.stl
- link MODULE_EE: geometry collision mesh filename=package://arm_description/meshes/Lower_leg_right.stl; visual mesh filename=package://arm_description/meshes/Lower_leg_right.stl

File: src/robot/arm_description/urdf/leg.urdf (robot description, URDF)
Before this commit: robot mulinex, 7 links, 6 joints
Links:
- link MODULE_1: geometry collision box size=0.269 0.057 0.060; visual mesh filename=package://arm_description/meshes/Module_right_front.stl
- link MODULE_2: geometry collision box size=0.269 0.057 0.060; visual mesh filename=package://arm_description/meshes/Module_right_front.stl
- link MODULE_3: geometry collision box size=0.269 0.057 0.060; visual mesh filename=package://arm_description/meshes/Module_right_front.stl
- link MODULE_EE: geometry collision mesh filename=package://arm_description/meshes/Lower_leg_right.stl; visual mesh filename=package://arm_description/meshes/Lower_leg_right.stl
