Commit message: Old changes

File: src/robot/arm_description/urdf/links.xacro (robot description, xacro)
@@ -121,4 +121,5 @@
                 <axis xyz="${axis}" />
                 <limit effort="2.7" lower="-${PI}" upper="${PI}" velocity="1000" />
+                <dynamics damping="0.0" friction="0.0"/>
             </joint>
         </xacro:unless>
@@ -137,4 +138,5 @@
             <axis xyz="${axis}" />
             <limit effort="2.7" lower="-${PI}" upper="${PI}" velocity="1000" />
+            <dynamics damping="0.0" friction="0.0"/>
         </joint>
         <!-- EE link -->
